File: MOSTERFET.kicad_pcb (KiCad board)
At the start: 2 copper layers, 50 x 60 mm, 32 parts, among them CN11 Jumper_NC_Small, CN21 Jumper_NC_Small, J11 XT-60, J12 XT-60, J21 XT-60, J22 XT-60, Q11 AUIRFSA8409-7P, Q21 AUIRFSA8409-7P, U11 TLP182, U21 TLP182

Commit message: Removed OSHW
Parts:
- moved REF*** 1.52 mm to (80.0, 87.0)
- moved H1 1.41 mm to (76.0, 87.0)
Other:
- board text removed: "OSHW xxxxx"
Changed lines of the file:
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@@
   (general
     (thickness 1.6)
-    (drawings 32)
+    (drawings 31)
     (tracks 162)
     (zones 0)
@@
     (aux_axis_origin 73 117)
     (grid_origin 73 117)
-    (visible_elements 7FFFF77F)
+    (visible_elements 7FFFE77F)
     (pcbplotparams
       (layerselection 0x010e0_ffffffff)
@@
   )
   (module Mounting_Holes:MountingHole_3.2mm_M3 (layer F.Cu)
-    (at 77 86)
+    (at 76 87)
     (descr "Mounting Hole 3.2mm, no annular, M3")
     (tags "mounting hole 3.2mm no annular m3")
@@
   )
   (module Symbols:OSHW-Symbol_8.9x8mm_SilkScreen (layer F.Cu)
-    (at 80.25 85.5)
+    (at 80 87)
     (descr "Open Source Hardware Symbol")
     (tags "Logo Symbol OSHW")
@@
     (effects (font (size 1.5 1.5) (thickness 0.3)) (justify left mirror))
   )
-  (gr_text "OSHW xxxxx" (at 80.75 90.75) (layer F.SilkS)
-    (effects (font (size 1.5 1.5) (thickness 0.3)))
-  )
   (gr_line (start 110.75 68) (end 102 68) (layer B.Mask) (width 5))
