File: Board Files/MOSTERFET.kicad_pcb (KiCad board)
At the start: 2 copper layers, 50 x 60 mm, 32 parts, among them CN11 Jumper_NC_Small, CN21 Jumper_NC_Small, J11 XT-60-M, J12 XT-60-F, J21 XT-60-M, J22 XT-60-F, Q11 AUIRFSA8409-7P, Q21 AUIRFSA8409-7P, U11 TLP182, U21 TLP182

Commit message: Added Bleed resistot
Parts:
- added R12: 10K, Resistors_SMD:R_1206_HandSoldering, F.Cu at (77.8, 88.2)
- added R22: 10K, Resistors_SMD:R_1206_HandSoldering, F.Cu at (77.9, 67.4)
Routing:
- net GND: track 21.3 -> 173.3 mm
- net Net-(D21-Pad3): track 6.96 -> 34.9 mm
- net Net-(D11-Pad3): track 6.58 -> 33.1 mm
